File: Main_Circuit/STLinkV3_Adapter.kicad_sch (KiCad schematic)
At the start: 10 parts, among them J1 Conn_01x03_Male, J2 Conn_01x05_Male, J3 Conn_01x04_Male, J4 Conn_01x05_Male, J5 Conn_01x04_Male, J6 Conn_01x06_Male, J7 Conn_01x06_Male, U1 STLINK-V3MODS

Commit message: Design PCB completed
Connections:
- net GND: no longer J1.1 (Pin_1), J2.1 (Pin_1), J3.1 (Pin_1), J4.1 (Pin_1), J5.1 (Pin_1)
- net GNDREF: now also J1.1 (Pin_1), J2.1 (Pin_1), J3.1 (Pin_1), J4.1 (Pin_1), J5.1 (Pin_1)
Changed lines of the file:
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@@
     (effects (font (size 1.27 1.27)) (justify left bottom))
   )
-  (label "GND" (at 177.165 101.5492 0)
+  (label "GNDREF" (at 177.165 101.5492 0)
     (effects (font (size 1.27 1.27)) (justify left bottom))
   )
@@
     (effects (font (size 1.27 1.27)) (justify right bottom))
   )
-  (label "GND" (at 144.5768 131.9784 0)
+  (label "GNDREF" (at 144.5768 131.9784 0)
     (effects (font (size 1.27 1.27)) (justify left bottom))
   )
@@
     (effects (font (size 1.27 1.27)) (justify left bottom))
   )
-  (label "GND" (at 144.78 101.8794 0)
+  (label "GNDREF" (at 144.78 101.8794 0)
     (effects (font (size 1.27 1.27)) (justify left bottom))
   )
@@
     (effects (font (size 1.27 1.27)) (justify right bottom))
   )
-  (label "GND" (at 181.102 132.08 0)
+  (label "GNDREF" (at 181.102 132.08 0)
     (effects (font (size 1.27 1.27)) (justify left bottom))
   )
@@
     (effects (font (size 1.27 1.27)) (justify right bottom))
   )
-  (label "GND" (at 206.6036 101.6 0)
+  (label "GNDREF" (at 206.6036 101.6 0)
     (effects (font (size 1.27 1.27)) (justify left bottom))
   )
